Commit message: Update

File: src/llm_robot/urdf/car_base.urdf (robot description, URDF)
Before this commit: robot car, 2 links, 1 joints
Links:
- added link caster_link; visual material name=black
- added link left_wheel_link; visual cylinder length=0.032 radius=0.04
- added link right_wheel_link; visual cylinder length=0.032 radius=0.04
- link camera_link: geometry visual box size=0.02 0.02 0.02
Joints:
- added joint caster_joint: type None, parent base_link, child caster_link, origin xyz=0.06 0.0 -0.076 rpy=0.0 0.0 0.0
- added joint left_wheel_joint: type continuous, parent base_link, child left_wheel_link, origin xyz=-0.02 0.10 -0.06 rpy=0.0 0.0 0.0, axis 0.0 1.0 0.0
- added joint right_wheel_joint: type continuous, parent base_link, child right_wheel_link, origin xyz=-0.02 -0.10 -0.06 rpy=0.0 0.0 0.0, axis 0.0 1.0 0.0

Commit message: Update

File: src/llm_robot/urdf/car_base.urdf (robot description, URDF)
Before this commit: robot car, 5 links, 4 joints
Links:
- added link base_footprint

Commit message: Update

File: src/llm_robot/urdf/car_base.urdf (robot description, URDF)
Before this commit: robot car, 6 links, 4 joints
Links:
- removed link base_footprint
- link caster_link: geometry visual box size=0.02 0.02 0.02
Joints:
- joint caster_joint: type None -> fixed
