Commit message: Supplement the missing mesh

File: src/robot_description/urdf/robot.xacro (robot description, xacro)
@@ -5,5 +5,5 @@
   xmlns:xacro="http://ros.org/wiki/xacro"
   name="sick_tim">
-  <xacro:include filename="$(find robot_sim_demo)/urdf/sick_tim.urdf.xacro" />
+  <xacro:include filename="$(find robot_description)/urdf/sick_tim.urdf.xacro" />
   <!-- Choose your laser -->
   <!--<xacro:sick_tim571 name="laser" ros_topic="scan"   />-->

File: src/robot_description/urdf/robot_dae.xacro (robot description, xacro)
@@ -5,11 +5,11 @@
   xmlns:xacro="http://ros.org/wiki/xacro"
   name="sick_tim">
-  <xacro:include filename="$(find robot_sim_demo)/urdf/sick_tim_dae.urdf.xacro" />
+  <xacro:include filename="$(find robot_description)/urdf/sick_tim_dae.urdf.xacro" />
   <!-- Choose your laser -->
   <!--<xacro:sick_tim571 name="laser" ros_topic="scan"   />-->
   <xacro:rplidarA2 name="laser" ros_topic="scan"   />
-  <xacro:include filename="$(find robot_sim_demo)/urdf/materials.xacro" />
-  <xacro:include filename="$(find robot_sim_demo)/urdf/xbot-u.urdf_dae.xacro" />
-  <xacro:include filename="$(find robot_sim_demo)/urdf/xbot-u.gazebo" />
+  <xacro:include filename="$(find robot_description)/urdf/materials.xacro" />
+  <xacro:include filename="$(find robot_description)/urdf/xbot-u.urdf_dae.xacro" />
+  <xacro:include filename="$(find robot_description)/urdf/xbot-u.gazebo" />
   <xacro:xbot2_base/>
 </robot>

File: src/robot_description/urdf/sick_tim.urdf.xacro (robot description, xacro)
@@ -8,5 +8,5 @@
       length="0.06" width="0.06" height="0.079" mass="0.150" z_offset="0.05595"
       min_range="0.2" max_range="8.0"
-      mesh="package://robot_sim_demo/models/meshes/rplidar.obj" />
+      mesh="package://robot_description/models/meshes/rplidar.obj" />
   </xacro:macro>
   <xacro:macro name="sick_tim310" params="name ros_topic">
@@ -14,5 +14,5 @@
       length="0.06" width="0.06" height="0.079" mass="0.150" z_offset="0.05595"
       min_range="0.05" max_range="4.0"
-      mesh="package://robot_sim_demo/models/meshes/sick_tim310.stl" />
+      mesh="package://robot_description/models/meshes/sick_tim310.stl" />
   </xacro:macro>
   <xacro:macro name="sick_tim551" params="name ros_topic">
@@ -20,5 +20,5 @@
       length="0.06" width="0.06" height="0.086" mass="0.250" z_offset="0.06296"
       min_range="0.05" max_range="10.0"
-      mesh="package://robot_sim_demo/models/meshes/sick_tim551.stl" />
+      mesh="package://robot_description/models/meshes/sick_tim551.stl" />
   </xacro:macro>
   <xacro:macro name="sick_tim571" params="name ros_topic">
@@ -26,5 +26,5 @@
       length="0.06" width="0.06" height="0.086" mass="0.250" z_offset="0.02"
       min_range="0.05" max_range="25.0"
-      mesh="package://robot_sim_demo/models/meshes/sick_tim571.stl" />
+      mesh="package://robot_description/models/meshes/sick_tim571.stl" />
   </xacro:macro>
   <xacro:macro name="sick_tim" params="name ros_topic length width height mass z_offset min_range max_range mesh">

File: src/robot_description/urdf/xbot-u.urdf.xacro (robot description, xacro)
@@ -21,5 +21,5 @@
       <origin xyz="0 0 0" rpy="0 0 0" />
       <geometry>
-        <mesh filename="package://robot_sim_demo/models/meshes/base_link.obj" />
+        <mesh filename="package://robot_description/models/meshes/base_link.obj" />
       </geometry>
     </visual>
@@ -85,5 +85,5 @@
       <origin xyz="0 0 0" rpy="0 0 -1.57079632"/>
       <geometry>
-        <mesh filename="package://robot_sim_demo/models/meshes/wheel.obj" />
+        <mesh filename="package://robot_description/models/meshes/wheel.obj" />
       </geometry>
     </visual>
@@ -112,5 +112,5 @@
       <origin xyz="0 0 0" rpy="0 0 1.57079632"/>
       <geometry>
-        <mesh filename="package://robot_sim_demo/models/meshes/wheel.obj" />
+        <mesh filename="package://robot_description/models/meshes/wheel.obj" />
       </geometry>
     </visual>
@@ -138,5 +138,5 @@
       <origin xyz="0 0 0" rpy="0 0 1.57079632" />
       <geometry>
-        <mesh filename="package://robot_sim_demo/models/meshes/yaw_platform.obj" />
+        <mesh filename="package://robot_description/models/meshes/yaw_platform.obj" />
       </geometry>
     </visual>
@@ -165,5 +165,5 @@
       <origin xyz="0 0 0" rpy="0 0 0" />
       <geometry>
-        <mesh filename="package://robot_sim_demo/models/meshes/pitch_platform.obj" />
+        <mesh filename="package://robot_description/models/meshes/pitch_platform.obj" />
       </geometry>
     </visual>
@@ -194,6 +194,6 @@
       <origin xyz="0 0 0" rpy="0 0 0"/>
       <geometry>
-        <!--<mesh filename="package://robot_sim_demo/models/meshes/xtion_pro_camera.dae" />-->
-        <mesh filename="package://robot_sim_demo/models/meshes/realsense.obj" />
+        <!--<mesh filename="package://robot_description/models/meshes/xtion_pro_camera.dae" />-->
+        <mesh filename="package://robot_description/models/meshes/realsense.obj" />
       </geometry>
     </visual>
