Commit message: Add gazebo plugin

File: src/robot_description/urdf/qpbot.xacro (robot description, xacro)
@@ -4,7 +4,149 @@
     <link name="base_footprint"/>
 	<xacro:include filename="./qpbot_components.xacro"/>
+	<!-- load components-->
     <xacro:create_base xyz_offset="0.0 0.0 0.076"/>
 	<xacro:create_wheel prefix="left" xyz_offset="-0.02 0.10 -0.06"/>
 	<xacro:create_wheel prefix="right" xyz_offset="-0.02 -0.10 -0.06"/>
 	<xacro:create_caster xyz_offset="0.06 0.0 -0.076"/>
+	<xacro:create_imu xyz_offset="0.0 0.0 0.02"/>
+	<xacro:create_laser xyz_offset="0.0 0.0 0.075"/>
+	<!-- gazebo settings -->
+	<!-- caster setting -->
+	<gazebo reference="caster_link">
+		<material>Gazebo/Black</material>
+		<mu1 value="0.0"/>
+		<mu2 value="0.0"/>
+		<kp value="1000000.0" />
+		<kd value="10.0" />
+	</gazebo>
+	<!-- wheel setting -->
+	<gazebo>
+		<plugin name="diff_drive" filename="libgazebo_ros_diff_drive.so">
+			<ros>
+				<namespace>/</namespace>
+				<remapping>cmd_vel:=cmd_vel</remapping>
+				<remapping>odom:=odom</remapping>
+			</ros>
+			<update_rate>30</update_rate>
+			<!-- whell-->
+			<left_joint>left_wheel_joint</left_joint>
+			<right_joint>right_wheel_joint</right_joint>
+			<!-- kinematics -->
+			<wheel_separation>0.2</wheel_separation>
+			<wheel_diameter>0.065</wheel_diameter>
+			<!-- limits -->
+			<max_wheel_torque>20</max_wheel_torque>
+			<max_wheel_acceleration>1.0</max_wheel_acceleration>
+			<!-- output -->
+			<publish_odom>true</publish_odom>
+			<publish_odom_tf>true</publish_odom_tf>
+			<publish_wheel_tf>true</publish_wheel_tf>
+			<odometry_frame>odom</odometry_frame>
+			<robot_base_frame>base_footprint</robot_base_frame>
+		</plugin>
+	</gazebo>
+	<!-- imu setting-->
+	<gazebo reference="imu_link">
+		<sensor name="imu_sensor" type="imu">
+			<plugin filename="libgazebo_ros_imu_sensor.so" name="imu_plugin">
+				<ros>
+					<namespace>/</namepsace>
+					<remapping>~/out:=imu</remapping>
+				</ros>
+				<initial_orientation_as_reference>flase</initial_orientation_as_reference>
+			</plugin>
+			<always_on>true</always_on>
+			<update_rate>100</update_rate>
+			<visualize>true</visualize>
+			<imu>
+				<angular_velocity>
+					<x>
+						<nosie type="gaussian">
+							<mean>0.0</mean>
+							<stddev>2e-4</stddev>
+                			<bias_mean>0.0000075</bias_mean>
+                			<bias_stddev>0.0000008</bias_stddev>
+						</noise>
+					</x>
+					<y>
+						<noise type="gaussian">
+							<mean>0.0</mean>
+							<stddev>2e-4</stddev>
+							<bias_mean>0.0000075</bias_mean>
+							<bias_stddev>0.0000008</bias_stddev>
+              			</noise>
+					</y>
+					<z>
+						<noise type="gaussian">
+							<mean>0.0</mean>
+							<stddev>2e-4</stddev>
+							<bias_mean>0.0000075</bias_mean>
+							<bias_stddev>0.0000008</bias_stddev>
+              			</noise>
+					</z>
+				</angular_velocity>
+				<linear_acceleration>
+					<x>
+              			<noise type="gaussian">
+							<mean>0.0</mean>
+							<stddev>1.7e-2</stddev>
+							<bias_mean>0.1</bias_mean>
+							<bias_stddev>0.001</bias_stddev>
+              			</noise>
+            		</x>
+					<y>
+              			<noise type="gaussian">
+							<mean>0.0</mean>
+							<stddev>1.7e-2</stddev>
+							<bias_mean>0.1</bias_mean>
+							<bias_stddev>0.001</bias_stddev>
+              			</noise>
+            		</y>
+					<z>
+              			<noise type="gaussian">
+							<mean>0.0</mean>
+							<stddev>1.7e-2</stddev>
+							<bias_mean>0.1</bias_mean>
+							<bias_stddev>0.001</bias_stddev>
+              			</noise>
+            		</z>
+				</linear_acceleration>
+			</imu>
+		</sensor>
+	</gazebo>
+	<!-- laser setting -->
+	<gazebo reference="laser_link">
+		<sensor name="laser_sensor" type="ray">
+			<always_on>true</always_on>
+			<visualize>trur</visualize>
+			<update_rate>10<update_rate>
+			<pose>0 0 0.075 0 0 0<pose>
+			<ray>
+				<scan>
+					<horizontal>
+						<samples>360</samples>
+						<resolution>1.000000</resolution>
+						<min_angle>0.000000</min_angle>
+						<max_angle>6.280000</max_angle>
+					</horizontal>
+				<scan>
+				<range>
+					<min>0.120000</min>
+					<max>3.500000</max>
+					<resolution>0.015000</resolution>
+				</range>
+				<noise type="gaussian">
+					<mean>0.0</mean>
+					<stddev>0.01</stddev>
+				</noise>
+			</ray>
+			<plugin name="laserscan" filename="libgazebo_ros_ray_sensor.so">
+				<ros>
+					<remapping>scan:=scan</remapping>
+				</ros>
+				<output_type>sensor_msgs/LaserScan</output_type>
+        		<frame_name>laser_link</frame_name>
+			</plugin>
+		</sensor>
+	</gazebo>
 </robot>

File: src/robot_description/urdf/qpbot_components.xacro (robot description, xacro)
@@ -141,5 +141,5 @@
     <xacro:macro name="create_laser" params="parent_link:=base_link xyz_offset:='0 0 0.02' rpy_offset:='0 0 0'">
         <!-- laser joint-->
-        <joint name="imu_joint" type="fixed">
+        <joint name="laser_joint" type="fixed">
             <parent link="${parent_link}"/>
             <child link="laser_link"/>
@@ -147,12 +147,12 @@
         </joint>
         <!-- laser link-->
-        <link name="imu_link">
+        <link name="laser_link">
             <visual>
                 <origin xyz="0 0 0" rpy="0 0 0"/>
                 <geometry>
-                    <box size="0.02 0.02 0.02"/>
+                    <cylinder radius="0.02" length="0.02"/>
                 </geometry>
                 <material name="black">
-                    <color rgba="0.0 0.0 0.0 0.0" />
+                    <color rgba="0.0 0.0 0.0 0.5" />
                 </material>
             </visual>
@@ -160,8 +160,8 @@
                 <origin xyz="0 0 0" rpy="0 0 0"/>
                 <geometry>
-                    <box size="0.02 0.02 0.02"/>
+                    <cylinder radius="0.02" length="0.02"/>
                 </geometry>
                 <material name="black">
-                    <color rgba="0.0 0.0 0.0 0.0" />
+                    <color rgba="0.0 0.0 0.0 0.5" />
                 </material>
             </collision>

Commit message: Fix launch error

File: src/robot_description/urdf/qpbot.xacro (robot description, xacro)
@@ -51,5 +51,5 @@
 			<plugin name="imu_plugin" filename="libgazebo_ros_imu_sensor.so" >
 				<ros>
-					<namespace>/</namepsace>
+					<namespace>/</namespace>
 					<remapping>~/out:=imu</remapping>
 				</ros>
@@ -120,6 +120,6 @@
 			<always_on>true</always_on>
 			<visualize>true</visualize>
-			<update_rate>10<update_rate>
-			<pose>0 0 0.075 0 0 0<pose>
+			<update_rate>10</update_rate>
+			<pose>0 0 0.075 0 0 0</pose>
 			<ray>
 				<scan>

File: src/robot_description/urdf/qpbot_components.xacro (robot description, xacro)
@@ -36,5 +36,5 @@
     </xacro:macro>
     <!-- wheel macro-->
-    <xacro:macro name="create_wheel" params="parent_link:=base_link prefix xyz_offset:='0 0 0' rpy_offset='0 0 0' axix=:'0 1 0'">
+    <xacro:macro name="create_wheel" params="parent_link:=base_link prefix xyz_offset:='0 0 0' rpy_offset='0 0 0' axis='0 1 0'">
         <!-- wheel joint -->
         <joint name="${prefix}_wheel_joint" type="continuous">
@@ -42,5 +42,5 @@
             <child link="${prefix}_wheel_link"/>
             <origin xyz="${xyz_offset}"/>
-            <axis xyz="${axix}"/>
+            <axis xyz="${axis}"/>
         </joint>
         <!-- wheel link -->
@@ -71,5 +71,5 @@
     </xacro:macro>
     <!-- caster marcro -->
-    <xacro:macro name="create_caster" params="parent_link:=base_link xyz_offset:='0 0 0' rpy_offset:='0 0 0' axix=:'0 1 0'">
+    <xacro:macro name="create_caster" params="parent_link:=base_link xyz_offset:='0 0 0' rpy_offset:='0 0 0' axis='0 1 0'">
         <!-- caster joint-->
         <joint name="caster_joint" type="fixed">
